File: KiCad/Sisyphus/Sisyphus.kicad_pcb (KiCad board)
At the start: 2 copper layers, 6 parts, among them SW1 SW_Push_SPDT, U1 ATmega328P-PU, Y1 Crystal

Commit message: adding a bunch of kicad stuff and references!
Parts:
- removed C1, C2: C, Capacitor_SMD:C_0603_1608Metric
- removed SW1: SW_Push_SPDT, Button_Switch_THT:SW_PUSH_6mm_H5mm
- removed Y1: Crystal, Crystal:Crystal_HC49-4H_Vertical
- added J1: Conn_01x07_Male, Connector_PinSocket_2.54mm:PinSocket_1x07_P2.54mm_Vertical, F.Cu at (264.0, 101.0)
- added J2: Conn_01x02_Male, Connector_PinSocket_2.54mm:PinSocket_1x02_P2.54mm_Vertical, F.Cu at (263.5, 79.5)
- added J3: Conn_01x04_Male, Connector_PinSocket_2.54mm:PinSocket_1x04_P2.54mm_Vertical, F.Cu at (263.5, 115.0)
- added R2: 2K, Resistor_SMD:R_0603_1608Metric_Pad1.05x0.95mm_HandSolder, F.Cu at (220.0, 100.2)
- added U2: MicroSD_Card_Adapter, Connector_PinHeader_2.54mm:PinHeader_1x06_P2.54mm_Vertical, F.Cu at (220.0, 102.8)
- added U3: TMC2130_Breakout, Sisyphus:TMC_2130_Footprint, F.Cu at (253.5, 89.5)
- added U4: TMC2130_Breakout, Sisyphus:TMC_2130_Footprint, F.Cu at (253.5, 111.0)
- R1: value R_US -> 2K
- U1: value ATmega328P-PU -> HUZZAH32; footprint Package_DIP:DIP-22_W7.62mm_Socket_LongPads -> Sisyphus:Huzzah32_Footprint
- moved U1 50.8 mm to (234.0, 99.0)
- moved R1 34.6 mm to (220.0, 97.7), turned to 0 degrees
Connections:
- R1 pad 1: +5V -> GND
- R1 pad 2: Net-(R1-Pad2) -> A3_39
- U1 pad 1: AT_PIN_1_RESET -> (no net)
- U1 pad 10: AT_PIN_10 -> A5_4
- U1 pad 11: Net-(U1-Pad11) -> SCK_5
- U1 pad 12: Net-(U1-Pad12) -> MOSI_18
- U1 pad 13: Net-(U1-Pad13) -> MISO_19
- U1 pad 14: Net-(U1-Pad14) -> (no net)
- U1 pad 15: Net-(U1-Pad15) -> (no net)
- U1 pad 16: Net-(U1-Pad16) -> 21
- U1 pad 17: Net-(U1-Pad17) -> (no net)
- U1 pad 18: Net-(U1-Pad18) -> (no net)
- U1 pad 19: Net-(U1-Pad19) -> A6_14
- U1 pad 2: Net-(U1-Pad2) -> 3V
- U1 pad 20: Net-(U1-Pad20) -> A7_32
- U1 pad 21: Net-(U1-Pad21) -> A8_15
- U1 pad 22: Earth -> A9_33
- U1 pad 3: Net-(U1-Pad3) -> (no net)
- U1 pad 4: Net-(U1-Pad4) -> GND
- U1 pad 5: Net-(U1-Pad5) -> (no net)
- U1 pad 6: Net-(U1-Pad6) -> (no net)
- U1 pad 7: +5V -> (no net)
- U1 pad 8: Earth -> A3_39
- U1 pad 9: AT_PIN_9 -> A4_36
Routing:
- net AT_PIN_9: track 30.8 -> 0.00 mm
- net AT_PIN_10: track 29.3 -> 0.00 mm
- net AT_PIN_1_RESET: track 19.8 -> 0.00 mm
- net +5V: track 15.6 -> 0.00 mm
- net Net-(R1-Pad2): track 15.6 -> 0.00 mm
- net Earth: track 12.0 -> 0.00 mm
Other:
- board outline added: 47.5 x 47.5 mm
