File: KiCad/Sisyphus/Sisyphus.sch (KiCad schematic (older format))
At the start: 9 parts, among them SW1 SW_Push_SPDT, U1 ATmega328P-PU, Y1 16Mhz

Commit message: adding a bunch of kicad stuff and references!
Parts:
- removed C1, C2: 22pF, Capacitor_SMD:C_0603_1608Metric, symbol Device:C
- removed J?: AVR-ISP-6, symbol Connector:AVR-ISP-6
- removed R1: 10K, Resistor_SMD:R_0603_1608Metric_Pad1.05x0.95mm_HandSolder, symbol Device:R_US
- removed SW1: SW_Push_SPDT, Button_Switch_THT:SW_PUSH_6mm_H5mm, symbol Switch:SW_Push_SPDT
- removed U1: ATmega328P-PU, Package_DIP:DIP-22_W7.62mm_Socket_LongPads, symbol MCU_Microchip_ATmega:ATmega328P-PU
- removed Y1: 16Mhz, Crystal:Crystal_HC49-4H_Vertical, symbol Device:Crystal
- added J1: Conn_01x07_Male, Connector_PinSocket_2.54mm:PinSocket_1x07_P2.54mm_Vertical, symbol Connector:Conn_01x07_Male
- added J2: Conn_01x02_Male, Connector_PinSocket_2.54mm:PinSocket_1x07_P2.54mm_Vertical, symbol Connector:Conn_01x02_Male
- added J3: Conn_01x04_Male, Connector_PinSocket_2.54mm:PinSocket_1x04_P2.54mm_Vertical, symbol Connector:Conn_01x04_Male
- added R1, R2: 2K, Resistor_SMD:R_0603_1608Metric_Pad1.05x0.95mm_HandSolder, symbol Device:R
- added U1: HUZZAH32, Sisyphus:Huzzah32_Footprint, symbol New_Library:HUZZAH32
- added U2: MicroSD_Card_Adapter, Connector_PinHeader_2.54mm:PinHeader_1x06_P2.54mm_Vertical, symbol New_Library:MicroSD_Card_Adapter
- U3, U4: renamed from U?; footprint (none) -> Sisyphus:TMC_2130_Footprint; symbol Driver_Motor:TMC2130_Breakout -> Sisyphus-rescue:TMC2130_Breakout-Driver_Motor
Connections:
- net labels added: 21, 3V, A10_27, A11_PDR_12, A12_13_LED, A3_39, A4_36, A5_4, A6_14, A7_32, A8_15, A9_33, GND, High_Motor_Voltage, Inner_Switch, MISO_19, MOSI_18, Outer_Switch, RX_16, Radius_Motor_A, Radius_Motor_B, Radius_Motor_C, Radius_Motor_D, SCK_5, SCL_22, SDA_23, TX_17, Theta_Motor_A, Theta_Motor_B, Theta_Motor_C, Theta_Motor_D, USB_5V
- net labels removed: +5V, AT_PIN_10, AT_PIN_16_SS, AT_PIN_17_MOSI, AT_PIN_18_MISO, AT_PIN_19_SCK, AT_PIN_1_RESET, AT_PIN_27_SDA_I2C, AT_PIN_28_SCL_I2C, AT_PIN_2_RX, AT_PIN_3_TX, AT_PIN_9, Earth
- wire segments 34 -> 8
- no-connect marks 0 -> 2
Other:
- note removed: "use these for sd cards and maybe tmc2130s\n"

Commit message: more kicad
Parts:
- J2: footprint Connector_PinSocket_2.54mm:PinSocket_1x07_P2.54mm_Vertical -> Connector_PinSocket_2.54mm:PinSocket_1x02_P2.54mm_Vertical
Changed lines of the file:
@@
 F 0 "J2" H 4008 5131 50  0000 C CNN
 F 1 "Conn_01x02_Male" H 4008 5040 50  0000 C CNN
-F 2 "Connector_PinSocket_2.54mm:PinSocket_1x07_P2.54mm_Vertical" H 3900 4950 50  0001 C CNN
+F 2 "Connector_PinSocket_2.54mm:PinSocket_1x02_P2.54mm_Vertical" H 3900 4950 50  0001 C CNN
 F 3 "~" H 3900 4950 50  0001 C CNN
 	1    3900 4950
